File: KiCad stuff/The Bomb Project/The Bomb Project.sch (KiCad schematic (older format))
At the start: 17 parts

Commit message: Use a demuxer and a single latch for simplicity
Parts:
- removed Q? (x8): Q_NMOS_GSD, symbol Device:Q_NMOS_GSD
- removed U? (x4): 74LS573, symbol 74xx:74LS573
- added Q1, Q2, Q3, Q4: MOSFET, Package_DIP:DIP-4_W7.62mm, symbol Device:Q_NMOS_GSD
- added R1, R2, R3, R4: 100, Resistor_THT:R_Axial_DIN0207_L6.3mm_D2.5mm_P10.16mm_Horizontal, symbol Device:R
- added U3: 74HC4051, symbol 74xx:74HC4051
- added U4: 74LS573, symbol 74xx:74LS573
- BZ1: renamed from BZ?; footprint (none) -> Connector_PinHeader_2.54mm:PinHeader_1x02_P2.54mm_Vertical
- J1: renamed from J?; footprint (none) -> Connector_PinHeader_2.54mm:PinHeader_2x03_P2.54mm_Vertical
- U1: renamed from U?; footprint (none) -> Package_TO_SOT_THT:TO-220-2_Horizontal_TabDown
- gave numbers to parts that had none: 2
Connections:
- wire segments 144 -> 51
- no-connect marks 0 -> 1
