File: KiCad stuff/The Bomb Project/The Bomb Project.sch (KiCad schematic (older format))
At the start: 9 parts

Commit message: Annotate case controller schematic
Parts:
- gave numbers to parts that had none: 9
Changed lines of the file:
@@
 $EndDescr
 $Comp
-L Connector_Generic:Conn_02x03_Odd_Even J?
+L Connector_Generic:Conn_02x03_Odd_Even J1
 U 1 1 5D7346A6
 P 1850 4000
-F 0 "J?" H 1850 4200 50  0000 R CNN
+F 0 "J1" H 1850 4200 50  0000 R CNN
 F 1 "ISP" H 2050 4200 50  0000 R CNN
 F 2 "" H 1850 4000 50  0001 C CNN
@@
 5v
 $Comp
-L power:Earth #PWR?
+L power:Earth #PWR0101
 U 1 1 5D74824F
 P 1650 4100
-F 0 "#PWR?" H 1650 3850 50  0001 C CNN
+F 0 "#PWR0101" H 1650 3850 50  0001 C CNN
 F 1 "Earth" H 1650 3950 50  0001 C CNN
 F 2 "" H 1650 4100 50  0001 C CNN
@@
 $EndComp
 $Comp
-L power:Earth #PWR?
+L power:Earth #PWR0102
 U 1 1 5D748395
 P 3350 5000
-F 0 "#PWR?" H 3350 4750 50  0001 C CNN
+F 0 "#PWR0102" H 3350 4750 50  0001 C CNN
 F 1 "Earth" H 3350 4850 50  0001 C CNN
 F 2 "" H 3350 5000 50  0001 C CNN
@@
 $EndComp
 $Comp
-L Regulator_Linear:L7805 U?
+L Regulator_Linear:L7805 U1
 U 1 1 5D74AD90
 P 1900 2700
-F 0 "U?" H 1750 2850 50  0000 C CNN
+F 0 "U1" H 1750 2850 50  0000 C CNN
 F 1 "L7805" H 2050 2850 50  0000 C CNN
 F 2 "" H 1925 2550 50  0001 L CIN
@@
 5v
 $Comp
-L power:Earth #PWR?
+L power:Earth #PWR0103
 U 1 1 5D74BAAF
 P 1900 3000
-F 0 "#PWR?" H 1900 2750 50  0001 C CNN
+F 0 "#PWR0103" H 1900 2750 50  0001 C CNN
 F 1 "Earth" H 1900 2850 50  0001 C CNN
 F 2 "" H 1900 3000 50  0001 C CNN
@@
 MOSI
 $Comp
-L Device:Buzzer BZ?
+L Device:Buzzer BZ1
 U 1 1 5D77FD04
 P 1850 3400
-F 0 "BZ?" H 2002 3429 50  0000 L CNN
+F 0 "BZ1" H 2002 3429 50  0000 L CNN
 F 1 "Buzzer" H 2002 3338 50  0000 L CNN
 F 2 "" V 1825 3500 50  0001 C CNN
@@
 $EndComp
 $Comp
-L power:Earth #PWR?
+L power:Earth #PWR0104
 U 1 1 5D780156
 P 1750 3500
-F 0 "#PWR?" H 1750 3250 50  0001 C CNN
+F 0 "#PWR0104" H 1750 3250 50  0001 C CNN
 F 1 "Earth" H 1750 3350 50  0001 C CNN
 F 2 "" H 1750 3500 50  0001 C CNN
@@
 CORRECT
 $Comp
-L The~Gelsoft~Bomb~Project:HDSP-B09G U?
+L The~Gelsoft~Bomb~Project:HDSP-B09G U4
 U 1 1 5D82E498
 P 9100 4550
-F 0 "U?" H 9100 5217 50  0000 C CNN
+F 0 "U4" H 9100 5217 50  0000 C CNN
 F 1 "HDSP-B09G" H 9100 5126 50  0000 C CNN
 F 2 "The Gelsoft Bomb Project:HDSP-B08G" H 9100 3950 50  0001 C CNN
@@
 5v
 $Comp
-L power:Earth #PWR?
+L power:Earth #PWR0105
 U 1 1 5D74EEF4
 P 6300 5250
-F 0 "#PWR?" H 6300 5000 50  0001 C CNN
+F 0 "#PWR0105" H 6300 5000 50  0001 C CNN
 F 1 "Earth" H 6300 5100 50  0001 C CNN
 F 2 "" H 6300 5250 50  0001 C CNN
@@
 $EndComp
 $Comp
-L The~Gelsoft~Bomb~Project:MAX7219 U?
+L The~Gelsoft~Bomb~Project:MAX7219 U3
 U 1 1 5D751E05
 P 6300 4300
-F 0 "U?" H 5900 5050 50  0000 C CNN
+F 0 "U3" H 5900 5050 50  0000 C CNN
 F 1 "MAX7219" H 6550 5050 50  0000 C CNN
 F 2 "" H 6350 5000 50  0001 C CNN
@@
 	6300 3400 7000 3400
 $Comp
-L Device:R R?
+L Device:R R1
 U 1 1 5D770D47
 P 7000 3550
-F 0 "R?" H 6930 3504 50  0000 R CNN
+F 0 "R1" H 6930 3504 50  0000 R CNN
 F 1 "20k" H 6930 3595 50  0000 R CNN
 F 2 "" V 6930 3550 50  0001 C CNN
@@
 	4900 4600 3950 4600
 $Comp
-L MCU_Microchip_ATtiny:ATtiny24A-PU U?
+L MCU_Microchip_ATtiny:ATtiny24A-PU U2
 U 1 1 5D807087
 P 3350 4100
-F 0 "U?" H 2950 4950 50  0000 R CNN
+F 0 "U2" H 2950 4950 50  0000 R CNN
 F 1 "ATtiny24A-PU" H 3950 4950 50  0000 R CNN
 F 2 "Package_DIP:DIP-14_W7.62mm" H 3350 4100 50  0001 C CIN
@@
 $EndComp
 $Comp
-L Connector:DB9_Male J?
+L Connector:DB9_Male J2
 U 1 1 5D86BF6C
 P 2000 5150
-F 0 "J?" H 1800 5750 50  0000 L CNN
+F 0 "J2" H 1800 5750 50  0000 L CNN
 F 1 "Module Connector" H 2000 5750 50  0000 L CNN
 F 2 "" H 2000 5150 50  0001 C CNN
@@
 LOWPOWER
 $Comp
-L power:Earth #PWR?
+L power:Earth #PWR0106
 U 1 1 5D8940BE
 P 1700 5550
-F 0 "#PWR?" H 1700 5300 50  0001 C CNN
+F 0 "#PWR0106" H 1700 5300 50  0001 C CNN
 F 1 "Earth" H 1700 5400 50  0001 C CNN
 F 2 "" H 1700 5550 50  0001 C CNN
@@
 $EndComp
 $Comp
-L Connector:Conn_01x02_Male J?
+L Connector:Conn_01x02_Male J3
 U 1 1 5D74C8FE
 P 2000 6150
-F 0 "J?" H 1972 6032 50  0000 R CNN
+F 0 "J3" H 1972 6032 50  0000 R CNN
 F 1 "Battery Header" H 1972 6123 50  0000 R CNN
 F 2 "" H 2000 6150 50  0001 C CNN
@@
 VIN
 $Comp
-L power:Earth #PWR?
+L power:Earth #PWR0107
 U 1 1 5D750EEE
 P 1800 6150
-F 0 "#PWR?" H 1800 5900 50  0001 C CNN
+F 0 "#PWR0107" H 1800 5900 50  0001 C CNN
 F 1 "Earth" H 1800 6000 50  0001 C CNN
 F 2 "" H 1800 6150 50  0001 C CNN

Commit message: Associate footprints with each component
Parts:
- BZ1, J3: footprint (none) -> Connector_PinHeader_2.54mm:PinHeader_1x02_P2.54mm_Vertical
- J1: footprint (none) -> Connector_PinHeader_2.54mm:PinHeader_2x03_P2.54mm_Vertical
- J2: footprint (none) -> Connector_Dsub:DSUB-9_Male_Horizontal_P2.77x2.84mm_EdgePinOffset4.94mm_Housed_MountingHolesOffset7.48mm
- R1: footprint (none) -> Resistor_THT:R_Axial_DIN0614_L14.3mm_D5.7mm_P20.32mm_Horizontal
- U1: footprint (none) -> Package_TO_SOT_THT:TO-220-4_Vertical
- U3: footprint (none) -> Package_DIP:DIP-24_W7.62mm
Changed lines of the file:
@@
 F 0 "J1" H 1850 4200 50  0000 R CNN
 F 1 "ISP" H 2050 4200 50  0000 R CNN
-F 2 "" H 1850 4000 50  0001 C CNN
+F 2 "Connector_PinHeader_2.54mm:PinHeader_2x03_P2.54mm_Vertical" H 1850 4000 50  0001 C CNN
 F 3 "~" H 1850 4000 50  0001 C CNN
 	1    1850 4000
@@
 F 0 "U1" H 1750 2850 50  0000 C CNN
 F 1 "L7805" H 2050 2850 50  0000 C CNN
-F 2 "" H 1925 2550 50  0001 L CIN
+F 2 "Package_TO_SOT_THT:TO-220-4_Vertical" H 1925 2550 50  0001 L CIN
 F 3 "http://www.st.com/content/ccc/resource/technical/document/datasheet/41/4f/b3/b0/12/d4/47/88/CD00000444.pdf/files/CD00000444.pdf/jcr:content/translations/en.CD00000444.pdf" H 1900 2650 50  0001 C CNN
 	1    1900 2700
@@
 F 0 "BZ1" H 2002 3429 50  0000 L CNN
 F 1 "Buzzer" H 2002 3338 50  0000 L CNN
-F 2 "" V 1825 3500 50  0001 C CNN
+F 2 "Connector_PinHeader_2.54mm:PinHeader_1x02_P2.54mm_Vertical" V 1825 3500 50  0001 C CNN
 F 3 "~" V 1825 3500 50  0001 C CNN
 	1    1850 3400
@@
 F 0 "U3" H 5900 5050 50  0000 C CNN
 F 1 "MAX7219" H 6550 5050 50  0000 C CNN
-F 2 "" H 6350 5000 50  0001 C CNN
+F 2 "Package_DIP:DIP-24_W7.62mm" H 6350 5000 50  0001 C CNN
 F 3 "" H 6350 5000 50  0001 C CNN
 	1    6300 4300
@@
 F 0 "R1" H 6930 3504 50  0000 R CNN
 F 1 "20k" H 6930 3595 50  0000 R CNN
-F 2 "" V 6930 3550 50  0001 C CNN
+F 2 "Resistor_THT:R_Axial_DIN0614_L14.3mm_D5.7mm_P20.32mm_Horizontal" V 6930 3550 50  0001 C CNN
 F 3 "~" H 7000 3550 50  0001 C CNN
 	1    7000 3550
@@
 F 0 "J2" H 1800 5750 50  0000 L CNN
 F 1 "Module Connector" H 2000 5750 50  0000 L CNN
-F 2 "" H 2000 5150 50  0001 C CNN
+F 2 "Connector_Dsub:DSUB-9_Male_Horizontal_P2.77x2.84mm_EdgePinOffset4.94mm_Housed_MountingHolesOffset7.48mm" H 2000 5150 50  0001 C CNN
 F 3 " ~" H 2000 5150 50  0001 C CNN
 	1    2000 5150
@@
 F 0 "J3" H 1972 6032 50  0000 R CNN
 F 1 "Battery Header" H 1972 6123 50  0000 R CNN
-F 2 "" H 2000 6150 50  0001 C CNN
+F 2 "Connector_PinHeader_2.54mm:PinHeader_1x02_P2.54mm_Vertical" H 2000 6150 50  0001 C CNN
 F 3 "~" H 2000 6150 50  0001 C CNN
 	1    2000 6150
