File: KiCad stuff/The Gelsoft Bomb Project/Module - Keypad.sch (KiCad schematic (older format))
At the start: 7 parts, among them J1 ISP, J2 Module Connector, U1 ATmega8-16PU, U2 74HC595, U3 3x4_Keypad, U4 SUR1601B

Commit message: Finalise the keypad module and add a PCB design
Parts:
- removed RV1: 10k, symbol Device:R_POT
- added R1: 10k, Resistor_THT:R_Axial_DIN0614_L14.3mm_D5.7mm_P20.32mm_Horizontal, symbol Device:R
- J2: footprint Connector_Dsub:DSUB-9_Male_Horizontal_P2.77x2.84mm_EdgePinOffset4.94mm_Housed_MountingHolesOffset7.48mm -> Connector_PinHeader_1.27mm:PinHeader_1x09_P1.27mm_Vertical
- U2: footprint (none) -> Package_DIP:DIP-16_W7.62mm
- U3: footprint (none) -> Connector_PinHeader_2.54mm:PinHeader_1x07_P2.54mm_Vertical
- U4: footprint (none) -> Connector_PinHeader_2.54mm:PinHeader_1x16_P2.54mm_Vertical
Changed lines of the file:
@@
 EESchema Schematic File Version 4
+LIBS:Module - Keypad-cache
 EELAYER 30 0
 EELAYER END
@@
 F 0 "J2" H 3100 5950 50  0000 L CNN
 F 1 "Module Connector" H 3300 5950 50  0000 L CNN
-F 2 "Connector_Dsub:DSUB-9_Male_Horizontal_P2.77x2.84mm_EdgePinOffset4.94mm_Housed_MountingHolesOffset7.48mm" H 3300 5350 50  0001 C CNN
+F 2 "Connector_PinHeader_1.27mm:PinHeader_1x09_P1.27mm_Vertical" H 3300 5350 50  0001 C CNN
 F 3 " ~" H 3300 5350 50  0001 C CNN
 	1    3300 5350
@@
 F 0 "U2" H 6800 2950 50  0000 C CNN
 F 1 "74HC595" H 7300 2950 50  0000 C CNN
-F 2 "" H 7050 2400 50  0001 C CNN
+F 2 "Package_DIP:DIP-16_W7.62mm" H 7050 2400 50  0001 C CNN
 F 3 "http://www.ti.com/lit/ds/symlink/sn74hc595.pdf" H 7050 2400 50  0001 C CNN
 	1    7050 2400
@@
 	8850 2000 8850 3700
 $Comp
-L Device:R_POT RV1
-U 1 1 5D81373A
-P 8150 3200
-F 0 "RV1" H 8000 3150 50  0000 C CNN
-F 1 "10k" H 8000 3250 50  0000 C CNN
-F 2 "" H 8150 3200 50  0001 C CNN
-F 3 "~" H 8150 3200 50  0001 C CNN
-	1    8150 3200
-	-1   0    0    1
-$EndComp
-$Comp
 L power:Earth #PWR0105
 U 1 1 5D814C30
@@
 	1    0    0    -1
 $EndComp
-Text GLabel 8000 3200 0    50   Input ~ 0
-5v
 Wire Wire Line
 	8150 3050 8150 2900
@@
 F 0 "U3" H 6750 5500 50  0000 L CNN
 F 1 "3x4_Keypad" H 7250 5500 50  0000 L CNN
-F 2 "" H 7050 5400 50  0001 C CNN
+F 2 "Connector_PinHeader_2.54mm:PinHeader_1x07_P2.54mm_Vertical" H 7050 5400 50  0001 C CNN
 F 3 "" H 7050 5400 50  0001 C CNN
 	1    7200 5000
@@
 F 0 "U4" H 7800 2850 50  0000 C CNN
 F 1 "SUR1601B" H 8350 2850 50  0000 C CNN
-F 2 "" H 7900 2550 50  0001 C CNN
+F 2 "Connector_PinHeader_2.54mm:PinHeader_1x16_P2.54mm_Vertical" H 7900 2550 50  0001 C CNN
 F 3 "https://ae01.alicdn.com/kf/HTB1vj1BmdcnBKNjSZR0q6AFqFXa9.jpg" H 7900 2550 50  0001 C CNN
 	1    8100 2350
@@
 Wire Wire Line
 	6150 3950 5600 3950
+$Comp
+L Device:R R1
+U 1 1 5DA19ACD
+P 8150 3200
+F 0 "R1" H 8220 3246 50  0000 L CNN
+F 1 "10k" H 8220 3155 50  0000 L CNN
+F 2 "Resistor_THT:R_Axial_DIN0614_L14.3mm_D5.7mm_P20.32mm_Horizontal" V 8080 3200 50  0001 C CNN
+F 3 "~" H 8150 3200 50  0001 C CNN
+	1    8150 3200
+	1    0    0    -1
+$EndComp
 $EndSCHEMATC
