File: KiCad stuff/The Gelsoft Bomb Project/Module - Keypad.sch (KiCad schematic (older format))
At the start: 7 parts, among them J1 ISP, J2 Module Connector, U1 ATmega8-16PU, U2 74HC595, U3 3x4_Keypad, U4 SUR1601B

Commit message: Add a new LCD and replace the old one
Parts:
- U4: value SUR1601B -> MC11605A6W7-BNMLW; symbol The~Gelsoft~Bomb~Project:SUR1601B -> The~Gelsoft~Bomb~Project:MC11605A6W7-BNMLW
Changed lines of the file:
@@
 $EndComp
 $Comp
-L The~Gelsoft~Bomb~Project:SUR1601B U4
+L The~Gelsoft~Bomb~Project:MC11605A6W7-BNMLW U4
 U 1 1 5D822D57
-P 8100 2350
-F 0 "U4" H 7800 2850 50  0000 C CNN
-F 1 "SUR1601B" H 8350 2850 50  0000 C CNN
-F 2 "Connector_PinHeader_2.54mm:PinHeader_1x16_P2.54mm_Vertical" H 7900 2550 50  0001 C CNN
-F 3 "https://ae01.alicdn.com/kf/HTB1vj1BmdcnBKNjSZR0q6AFqFXa9.jpg" H 7900 2550 50  0001 C CNN
-	1    8100 2350
+P 8150 1900
+F 0 "U4" H 7800 1950 50  0000 C CNN
+F 1 "MC11605A6W7-BNMLW" H 8600 1950 50  0000 C CNN
+F 2 "Connector_PinHeader_2.54mm:PinHeader_1x16_P2.54mm_Vertical" H 7950 2100 50  0001 C CNN
+F 3 "https://ae01.alicdn.com/kf/HTB1vj1BmdcnBKNjSZR0q6AFqFXa9.jpg" H 7950 2100 50  0001 C CNN
+	1    8150 1900
 	1    0    0    -1
 $EndComp

Commit message: Update keypad with new connector pinout
Parts:
- U1: symbol MCU_Microchip_ATmega:ATmega8-16PU -> Module---Keypad-rescue:ATmega8-16PU-MCU_Microchip_ATmega
Connections:
- net labels removed: CORRECT, DISARM, LOWPOWER, STRIKE
- wire segments 54 -> 62
Other:
- moved on the sheet: R1
Changed lines of the file:
@@
 EESchema Schematic File Version 4
-LIBS:Module - Keypad-cache
 EELAYER 30 0
 EELAYER END
@@
 Text GLabel 5600 3750 2    50   Input ~ 0
 SCK
-Text GLabel 5600 3350 2    50   Output ~ 0
-STRIKE
-Text GLabel 5600 3450 2    50   Input ~ 0
-DISARM
 Text GLabel 5600 3550 2    50   Input ~ 0
 MOSI
-Text GLabel 4400 3450 0    50   Input ~ 0
-LOWPOWER
-Text GLabel 5600 3250 2    50   Output ~ 0
-CORRECT
 $Comp
 L Connector:DB9_Female J2
@@
 	1    0    0    -1
 $EndComp
-Text GLabel 3000 4950 0    50   Output ~ 0
-5v
-Text GLabel 3000 5650 0    50   Input ~ 0
-CORRECT
-Text GLabel 3000 5450 0    50   Input ~ 0
-STRIKE
-Text GLabel 3000 5250 0    50   Output ~ 0
-DISARM
-Text GLabel 3000 5050 0    50   Output ~ 0
-LOWPOWER
+Text GLabel 3000 5650 0    50   Output ~ 0
+5v
+Text GLabel 3000 5750 0    50   Output ~ 0
+SCK
+Text GLabel 3000 5350 0    50   Input ~ 0
+MOSI
+Text GLabel 3000 5550 0    50   Output ~ 0
+MISO
 $Comp
 L power:Earth #PWR0106
 U 1 1 5D8940BE
-P 3000 5750
-F 0 "#PWR0106" H 3000 5500 50  0001 C CNN
-F 1 "Earth" H 3000 5600 50  0001 C CNN
-F 2 "" H 3000 5750 50  0001 C CNN
-F 3 "~" H 3000 5750 50  0001 C CNN
-	1    3000 5750
-	1    0    0    -1
-$EndComp
-Text GLabel 3000 5150 0    50   Output ~ 0
+P 2900 5150
+F 0 "#PWR0106" H 2900 4900 50  0001 C CNN
+F 1 "Earth" H 2900 5000 50  0001 C CNN
+F 2 "" H 2900 5150 50  0001 C CNN
+F 3 "~" H 2900 5150 50  0001 C CNN
+	1    2900 5150
+	1    0    0    -1
+$EndComp
+Text GLabel 3000 5450 0    50   Output ~ 0
 VIN
 $Comp
@@
 	1    0    0    -1
 $EndComp
-$Comp
-L power:Earth #PWR0104
-U 1 1 5D80FA51
-P 8050 2900
-F 0 "#PWR0104" H 8050 2650 50  0001 C CNN
-F 1 "Earth" H 8050 2750 50  0001 C CNN
-F 2 "" H 8050 2900 50  0001 C CNN
-F 3 "~" H 8050 2900 50  0001 C CNN
-	1    8050 2900
-	1    0    0    -1
-$EndComp
 Text GLabel 7050 1800 1    50   Input ~ 0
 5v
@@
 $EndComp
 Wire Wire Line
-	8150 3050 8150 2900
+	8150 2950 8150 2900
 $Comp
 L The~Gelsoft~Bomb~Project:3x4_Keypad U3
@@
 $EndComp
 $Comp
-L MCU_Microchip_ATmega:ATmega8-16PU U1
+L Module---Keypad-rescue:ATmega8-16PU-MCU_Microchip_ATmega U1
 U 1 1 5D825400
 P 5000 4350
@@
 	6300 3550 8700 3550
 Wire Wire Line
-	4400 3650 3850 3650
-Wire Wire Line
-	3850 3650 3850 2300
-Wire Wire Line
-	3850 2300 6650 2300
+	4400 3650 4050 3650
+Wire Wire Line
+	4050 3650 4050 2300
+Wire Wire Line
+	4050 2300 6650 2300
 Wire Wire Line
 	5600 4150 6250 4150
@@
 L Device:R R1
 U 1 1 5DA19ACD
-P 8150 3200
-F 0 "R1" H 8220 3246 50  0000 L CNN
-F 1 "10k" H 8220 3155 50  0000 L CNN
-F 2 "Resistor_THT:R_Axial_DIN0614_L14.3mm_D5.7mm_P20.32mm_Horizontal" V 8080 3200 50  0001 C CNN
-F 3 "~" H 8150 3200 50  0001 C CNN
-	1    8150 3200
+P 8150 3100
+F 0 "R1" H 8220 3146 50  0000 L CNN
+F 1 "10k" H 8220 3055 50  0000 L CNN
+F 2 "Resistor_THT:R_Axial_DIN0614_L14.3mm_D5.7mm_P20.32mm_Horizontal" V 8080 3100 50  0001 C CNN
+F 3 "~" H 8150 3100 50  0001 C CNN
+	1    8150 3100
 	1    0    0    -1
 $EndComp
@@
 Text Notes 5250 4400 2    50   ~ 0
 LCD Mode/LED
+Wire Wire Line
+	3000 4950 3000 5050
+Wire Wire Line
+	3000 5050 3000 5150
+Connection ~ 3000 5050
+Wire Wire Line
+	3000 5150 3000 5250
+Connection ~ 3000 5150
+Wire Wire Line
+	2900 5150 3000 5150
+Wire Wire Line
+	8050 2900 8050 3300
+Wire Wire Line
+	8050 3300 8150 3300
+Wire Wire Line
+	8150 3300 8150 3350
+Wire Wire Line
+	8150 3300 8150 3250
+Connection ~ 8150 3300
 $EndSCHEMATC

Commit message: Use better footprints
Parts:
- J2: footprint Connector_PinHeader_1.27mm:PinHeader_1x09_P1.27mm_Vertical -> Connector_IDC:IDC-Header_2x05_P2.54mm_Vertical
- R1: footprint Resistor_THT:R_Axial_DIN0614_L14.3mm_D5.7mm_P20.32mm_Horizontal -> Resistor_THT:R_Axial_DIN0207_L6.3mm_D2.5mm_P10.16mm_Horizontal
- U1: symbol Module---Keypad-rescue:ATmega8-16PU-MCU_Microchip_ATmega -> MCU_Microchip_ATmega:ATmega8-16PU
- U3: footprint Connector_PinHeader_2.54mm:PinHeader_1x07_P2.54mm_Vertical -> Connector_IDC:IDC-Header_2x04_P2.54mm_Vertical
Changed lines of the file:
@@
 F 0 "J2" H 3100 5950 50  0000 L CNN
 F 1 "Module Connector" H 3300 5950 50  0000 L CNN
-F 2 "Connector_PinHeader_1.27mm:PinHeader_1x09_P1.27mm_Vertical" H 3300 5350 50  0001 C CNN
+F 2 "Connector_IDC:IDC-Header_2x05_P2.54mm_Vertical" H 3300 5350 50  0001 C CNN
 F 3 " ~" H 3300 5350 50  0001 C CNN
 	1    3300 5350
@@
 F 0 "U3" H 6750 5500 50  0000 L CNN
 F 1 "3x4_Keypad" H 7250 5500 50  0000 L CNN
-F 2 "Connector_PinHeader_2.54mm:PinHeader_1x07_P2.54mm_Vertical" H 7050 5400 50  0001 C CNN
+F 2 "Connector_IDC:IDC-Header_2x04_P2.54mm_Vertical" H 7050 5400 50  0001 C CNN
 F 3 "" H 7050 5400 50  0001 C CNN
 	1    7200 5000
@@
 $EndComp
 $Comp
-L Module---Keypad-rescue:ATmega8-16PU-MCU_Microchip_ATmega U1
+L MCU_Microchip_ATmega:ATmega8-16PU U1
 U 1 1 5D825400
 P 5000 4350
@@
 F 0 "R1" H 8220 3146 50  0000 L CNN
 F 1 "10k" H 8220 3055 50  0000 L CNN
-F 2 "Resistor_THT:R_Axial_DIN0614_L14.3mm_D5.7mm_P20.32mm_Horizontal" V 8080 3100 50  0001 C CNN
+F 2 "Resistor_THT:R_Axial_DIN0207_L6.3mm_D2.5mm_P10.16mm_Horizontal" V 8080 3100 50  0001 C CNN
 F 3 "~" H 8150 3100 50  0001 C CNN
 	1    8150 3100
