File: KiCad stuff/The Gelsoft Bomb Project/Case Controller.sch (KiCad schematic (older format))
At the start: 9 parts, among them J1 ISP, J2 Module Connector, J3 Battery Header, U1 L7805, U2 ATtiny24A-PU, U3 MAX7219, U4 HDSP-B09G

Commit message: Add decoupling cap to the MAX7219
It makes an unbearable noise on the buzzer if left untreated
Parts:
- added C1: 0.1uF, Capacitor_THT:C_Axial_L5.1mm_D3.1mm_P10.00mm_Horizontal, symbol Device:C
Connections:
- wire segments 46 -> 49
Changed lines of the file:
@@
 EESchema Schematic File Version 4
-LIBS:The Bomb Project-cache
 EELAYER 30 0
 EELAYER END
@@
 Wire Wire Line
 	8000 4250 6850 4250
-Text GLabel 6300 3350 1    50   Input ~ 0
+Text GLabel 6300 3050 1    50   Input ~ 0
 5v
 $Comp
@@
 	-1   0    0    1
 $EndComp
-Wire Wire Line
-	6300 3400 6300 3350
 Connection ~ 6300 3400
 Wire Wire Line
@@
 	1    0    0    -1
 $EndComp
+$Comp
+L Device:C C1
+U 1 1 5DC04291
+P 6150 3200
+F 0 "C1" V 6000 3200 50  0000 C CNN
+F 1 "0.1uF" V 6300 3200 50  0000 C CNN
+F 2 "Capacitor_THT:C_Axial_L5.1mm_D3.1mm_P10.00mm_Horizontal" H 6188 3050 50  0001 C CNN
+F 3 "~" H 6150 3200 50  0001 C CNN
+	1    6150 3200
+	0    1    1    0
+$EndComp
+Wire Wire Line
+	6300 3050 6300 3200
+Wire Wire Line
+	6300 3200 6300 3400
+Connection ~ 6300 3200
+$Comp
+L power:Earth #PWR0108
+U 1 1 5DC0839B
+P 5950 3250
+F 0 "#PWR0108" H 5950 3000 50  0001 C CNN
+F 1 "Earth" H 5950 3100 50  0001 C CNN
+F 2 "" H 5950 3250 50  0001 C CNN
+F 3 "~" H 5950 3250 50  0001 C CNN
+	1    5950 3250
+	1    0    0    -1
+$EndComp
+Wire Wire Line
+	5950 3250 5950 3200
+Wire Wire Line
+	5950 3200 6000 3200
 $EndSCHEMATC

Commit message: Board tweaks
Parts:
- removed C1: 0.1uF, Capacitor_THT:C_Axial_L5.1mm_D3.1mm_P10.00mm_Horizontal, symbol Device:C
- added C1: 100uF, Capacitor_THT:CP_Radial_D6.3mm_P2.50mm, symbol Device:CP
- R1: footprint Resistor_THT:R_Axial_DIN0614_L14.3mm_D5.7mm_P20.32mm_Horizontal -> Resistor_THT:R_Axial_DIN0207_L6.3mm_D2.5mm_P10.16mm_Horizontal
Changed lines of the file:
@@
 Wire Wire Line
 	8000 4250 6850 4250
-Text GLabel 6300 3050 1    50   Input ~ 0
+Text GLabel 6300 2900 1    50   Input ~ 0
 5v
 $Comp
@@
 F 0 "R1" H 6930 3504 50  0000 R CNN
 F 1 "20k" H 6930 3595 50  0000 R CNN
-F 2 "Resistor_THT:R_Axial_DIN0614_L14.3mm_D5.7mm_P20.32mm_Horizontal" V 6930 3550 50  0001 C CNN
+F 2 "Resistor_THT:R_Axial_DIN0207_L6.3mm_D2.5mm_P10.16mm_Horizontal" V 6930 3550 50  0001 C CNN
 F 3 "~" H 7000 3550 50  0001 C CNN
 	1    7000 3550
@@
 $EndComp
 $Comp
-L Device:C C1
-U 1 1 5DC04291
-P 6150 3200
-F 0 "C1" V 6000 3200 50  0000 C CNN
-F 1 "0.1uF" V 6300 3200 50  0000 C CNN
-F 2 "Capacitor_THT:C_Axial_L5.1mm_D3.1mm_P10.00mm_Horizontal" H 6188 3050 50  0001 C CNN
-F 3 "~" H 6150 3200 50  0001 C CNN
-	1    6150 3200
+L power:Earth #PWR0108
+U 1 1 5DD711D2
+P 5900 3200
+F 0 "#PWR0108" H 5900 2950 50  0001 C CNN
+F 1 "Earth" H 5900 3050 50  0001 C CNN
+F 2 "" H 5900 3200 50  0001 C CNN
+F 3 "~" H 5900 3200 50  0001 C CNN
+	1    5900 3200
+	1    0    0    -1
+$EndComp
+$Comp
+L Device:CP C1
+U 1 1 5DD72109
+P 6050 3150
+F 0 "C1" V 5900 3050 50  0000 C CNN
+F 1 "100uF" V 5900 3250 50  0000 C CNN
+F 2 "Capacitor_THT:CP_Radial_D6.3mm_P2.50mm" H 6088 3000 50  0001 C CNN
+F 3 "~" H 6050 3150 50  0001 C CNN
+	1    6050 3150
 	0    1    1    0
 $EndComp
 Wire Wire Line
-	6300 3050 6300 3200
-Wire Wire Line
-	6300 3200 6300 3400
-Connection ~ 6300 3200
-$Comp
-L power:Earth #PWR0108
-U 1 1 5DC0839B
-P 5950 3250
-F 0 "#PWR0108" H 5950 3000 50  0001 C CNN
-F 1 "Earth" H 5950 3100 50  0001 C CNN
-F 2 "" H 5950 3250 50  0001 C CNN
-F 3 "~" H 5950 3250 50  0001 C CNN
-	1    5950 3250
-	1    0    0    -1
-$EndComp
-Wire Wire Line
-	5950 3250 5950 3200
-Wire Wire Line
-	5950 3200 6000 3200
+	5900 3200 5900 3150
+Wire Wire Line
+	6300 2900 6300 3150
+Wire Wire Line
+	6200 3150 6300 3150
+Connection ~ 6300 3150
+Wire Wire Line
+	6300 3150 6300 3400
 $EndSCHEMATC

Commit message: Revise case controller
Added a buck converter for more efficient power regulation
Added a diode to the battery for safety
Added a power switch
Reworked the PCB design to suit these upgrades
Parts:
- removed U1: L7805, Package_TO_SOT_THT:TO-220-4_Vertical, symbol Regulator_Linear:L7805
- added D1: 1N5400, Diode_THT:D_DO-201AD_P15.24mm_Horizontal, symbol Device:D
- added SW1: Power Switch, The Gelsoft Bomb Project:SK12D07VG3, symbol Switch:SW_SPST
- C1: value 100uF -> 470uF; footprint Capacitor_THT:CP_Radial_D6.3mm_P2.50mm -> Capacitor_THT:CP_Radial_D10.0mm_P5.00mm
Connections:
- wire segments 49 -> 52
Changed lines of the file:
@@
 EESchema Schematic File Version 4
+LIBS:Case Controller-cache
 EELAYER 30 0
 EELAYER END
 $Descr A4 11693 8268
 encoding utf-8
-Sheet 1 1
+Sheet 1 2
 Title "Gelsoft Bomb Poject Case Controller"
 Date ""
@@
 	1    0    0    -1
 $EndComp
-$Comp
-L Regulator_Linear:L7805 U1
-U 1 1 5D74AD90
-P 1900 2700
-F 0 "U1" H 1750 2850 50  0000 C CNN
-F 1 "L7805" H 2050 2850 50  0000 C CNN
-F 2 "Package_TO_SOT_THT:TO-220-4_Vertical" H 1925 2550 50  0001 L CIN
-F 3 "http://www.st.com/content/ccc/resource/technical/document/datasheet/41/4f/b3/b0/12/d4/47/88/CD00000444.pdf/files/CD00000444.pdf/jcr:content/translations/en.CD00000444.pdf" H 1900 2650 50  0001 C CNN
-	1    1900 2700
-	1    0    0    -1
-$EndComp
 Text GLabel 1600 2700 0    50   Input ~ 0
 VIN
-Text GLabel 2200 2700 2    50   Output ~ 0
-5v
-$Comp
-L power:Earth #PWR0103
-U 1 1 5D74BAAF
-P 1900 3000
-F 0 "#PWR0103" H 1900 2750 50  0001 C CNN
-F 1 "Earth" H 1900 2850 50  0001 C CNN
-F 2 "" H 1900 3000 50  0001 C CNN
-F 3 "~" H 1900 3000 50  0001 C CNN
-	1    1900 3000
-	1    0    0    -1
-$EndComp
+Text GLabel 1600 2800 0    50   Output ~ 0
+5v
 Text GLabel 3950 4000 2    50   Output ~ 0
 MISO
@@
 L Connector:Conn_01x02_Male J3
 U 1 1 5D74C8FE
-P 2000 6150
-F 0 "J3" H 1972 6032 50  0000 R CNN
-F 1 "Battery Header" H 1972 6123 50  0000 R CNN
-F 2 "Connector_PinHeader_2.54mm:PinHeader_1x02_P2.54mm_Vertical" H 2000 6150 50  0001 C CNN
-F 3 "~" H 2000 6150 50  0001 C CNN
-	1    2000 6150
+P 2500 6200
+F 0 "J3" H 2472 6082 50  0000 R CNN
+F 1 "Battery Header" H 2472 6173 50  0000 R CNN
+F 2 "Connector_PinHeader_2.54mm:PinHeader_1x02_P2.54mm_Vertical" H 2500 6200 50  0001 C CNN
+F 3 "~" H 2500 6200 50  0001 C CNN
+	1    2500 6200
 	-1   0    0    1
 $EndComp
 Text GLabel 1700 4950 0    50   BiDi ~ 0
 VIN
-Text GLabel 1800 6050 0    50   Output ~ 0
+Text GLabel 1200 6100 0    50   Output ~ 0
 VIN
 $Comp
 L power:Earth #PWR0107
 U 1 1 5D750EEE
-P 1800 6150
-F 0 "#PWR0107" H 1800 5900 50  0001 C CNN
-F 1 "Earth" H 1800 6000 50  0001 C CNN
-F 2 "" H 1800 6150 50  0001 C CNN
-F 3 "~" H 1800 6150 50  0001 C CNN
-	1    1800 6150
+P 2300 6200
+F 0 "#PWR0107" H 2300 5950 50  0001 C CNN
+F 1 "Earth" H 2300 6050 50  0001 C CNN
+F 2 "" H 2300 6200 50  0001 C CNN
+F 3 "~" H 2300 6200 50  0001 C CNN
+	1    2300 6200
 	1    0    0    -1
 $EndComp
@@
 P 6050 3150
 F 0 "C1" V 5900 3050 50  0000 C CNN
-F 1 "100uF" V 5900 3250 50  0000 C CNN
-F 2 "Capacitor_THT:CP_Radial_D6.3mm_P2.50mm" H 6088 3000 50  0001 C CNN
+F 1 "470uF" V 5900 3250 50  0000 C CNN
+F 2 "Capacitor_THT:CP_Radial_D10.0mm_P5.00mm" H 6088 3000 50  0001 C CNN
 F 3 "~" H 6050 3150 50  0001 C CNN
 	1    6050 3150
@@
 Wire Wire Line
 	6300 3150 6300 3400
+$Sheet
+S 1600 2600 550  300
+U 5DE64F8A
+F0 "Buck Converter" 50
+F1 "Buck Converter.sch" 50
+F2 "VIN" I L 1600 2700 50
+F3 "VOUT" O L 1600 2800 50
+$EndSheet
+$Comp
+L Switch:SW_SPST SW1
+U 1 1 5DE69AC5
+P 2050 6100
+F 0 "SW1" H 2050 6300 50  0000 C CNN
+F 1 "Power Switch" H 2050 6200 50  0000 C CNN
+F 2 "The Gelsoft Bomb Project:SK12D07VG3" H 2050 6100 50  0001 C CNN
+F 3 "~" H 2050 6100 50  0001 C CNN
+	1    2050 6100
+	1    0    0    -1
+$EndComp
+Wire Wire Line
+	2250 6100 2300 6100
+Wire Wire Line
+	1850 6100 1600 6100
+$Comp
+L Device:D D1
+U 1 1 5DE00C5D
+P 1450 6100
+F 0 "D1" H 1450 6300 50  0000 C CNN
+F 1 "1N5400" H 1450 6200 50  0000 C CNN
+F 2 "Diode_THT:D_DO-201AD_P15.24mm_Horizontal" H 1450 6100 50  0001 C CNN
+F 3 "~" H 1450 6100 50  0001 C CNN
+	1    1450 6100
+	1    0    0    -1
+$EndComp
+Wire Wire Line
+	1200 6100 1300 6100
 $EndSCHEMATC

Commit message: Overhaul into v0.2.0 (see desc)
Added buttons to set the timer
Added the low-power switch
Added strike LEDs (2 for now, since we don't want another LED driver)
Parts:
- added D2: STRIKE 1, The Gelsoft Bomb Project:LED_Square_15x15mm, symbol Device:LED
- added D3: STRIKE 2, The Gelsoft Bomb Project:LED_Square_15x15mm, symbol Device:LED
- added J4: Low-Power Switch, Connector_PinHeader_2.54mm:PinHeader_1x02_P2.54mm_Vertical, symbol Connector:Conn_01x02_Male
- added R5, R6, R7, R8: 100k, Resistor_THT:R_Axial_DIN0207_L6.3mm_D2.5mm_P10.16mm_Horizontal, symbol Device:R
- added SW2: PLUS, Button_Switch_THT:SW_PUSH_6mm, symbol Switch:SW_SPST
- added SW3: MINUS, Button_Switch_THT:SW_PUSH_6mm, symbol Switch:SW_SPST
- added SW4: OK, Button_Switch_THT:SW_PUSH_6mm, symbol Switch:SW_SPST
Connections:
- net labels added: MINUS, OK, PLUS
- net labels removed: CORRECT, DISARM, STRIKE
- wire segments 52 -> 81
Other:
- moved on the sheet: J1

Commit message: Replace buck converter with a pre-made module
Bugger having to deal with making my own, we'll just keep things simple and cheap
Parts:
- added U1: Buck_Converter_Module_7-26v, The Gelsoft Bomb Project:Buck_Converter_Module_7-24v, symbol The~Gelsoft~Bomb~Project:Buck_Converter_Module_7-26v
Connections:
- wire segments 81 -> 84
Other:
- moved on the sheet: J1, R5, R6, R7, R8
